Commit message: 小料坏

File: rm_robot_description/urdf/rm_gimbal.urdf.xacro (robot description, xacro)
@@ -4,8 +4,8 @@
   <xacro:arg name="xyz" default="0.10 0 0.05" />
   <xacro:arg name="rpy" default="0 0 0" />
-  <link name="odom" />
+  <link name="gimbal_odom" />
   <link name="gimbal_link" />
   <joint name="gimbal_joint" type="floating">
-    <parent link="odom" />
+    <parent link="gimbal_odom" />
     <child link="gimbal_link" />
   </joint>

Commit message: 小料坏！！！

File: rm_robot_description/urdf/rm_gimbal.urdf.xacro (robot description, xacro)
@@ -4,8 +4,8 @@
   <xacro:arg name="xyz" default="0.10 0 0.05" />
   <xacro:arg name="rpy" default="0 0 0" />
-  <link name="gimbal_odom" />
+  <link name="odom" />
   <link name="gimbal_link" />
   <joint name="gimbal_joint" type="floating">
-    <parent link="gimbal_odom" />
+    <parent link="odom" />
     <child link="gimbal_link" />
   </joint>
